Commit message: Add files via upload
finally working combined model in gazebo

File: gantry_robot_hvl/urdf/gantry_v1.urdf.xacro (robot description, xacro)
@@ -6,22 +6,28 @@
     <parent link="world"/>
     <child link="left_support_arch_link" />
-    <origin xyz="5.5 0 0" rpy="0 0 0"/>
+    <origin xyz="2.6 0 0" rpy="0 0 0"/>
   </joint>
   <joint name="world_joint_right" type="fixed">
     <parent link="world"/>
     <child link="right_support_arch_link" />
-    <origin xyz="-5.5 0 0" rpy="0 0 0"/>
-  </joint>
-  <!--Support_arch left side -->
-  <xacro:property name="support_arch_length" value="10" />
-  <xacro:property name="support_arch_width" value="1" />
+    <origin xyz="-2.6 0 0" rpy="0 0 0"/>
+  </joint>
+  <xacro:property name="support_scale_x" value= "0.0005" />
+  <xacro:property name="support_scale_y" value= "0.0005" />
+  <xacro:property name="support_scale_z" value= "0.00075" />
+  <xacro:property name="high_scale" value= "0.0005" />
+  <xacro:property name="mid_scale" value= "0.005" />
+  <xacro:property name="low_scale" value= "0.5" />
+  <xacro:property name="support_arch_length" value="5" />
+  <xacro:property name="support_arch_width" value="0.5" />
   <xacro:property name="support_arch_height" value="3.3" />
   <xacro:property name="support_arch_density" value="1" />
   <xacro:property name="support_arch_mass" value="${support_arch_length*support_arch_height*support_arch_width*support_arch_density}" />
+    <!--Support_arch left side -->
   <link name="left_support_arch_link">
     <visual>
       <origin  rpy="0 0 0" xyz="0 0 0"/>
       <geometry>
-        <mesh filename="package://gantry_robot_hvl/meshes/support_arch_v2.stl" scale="0.001 0.001 0.001"/>
+        <mesh filename="package://gantry_robot_hvl/meshes/support_arch_v2.stl" scale="${support_scale_x} ${support_scale_y} ${support_scale_z}"/>
       </geometry>
     </visual>
@@ -46,5 +52,5 @@
         <origin xyz="0 0 0" rpy="0 0 0"/>
         <geometry>
-          <mesh filename="package://gantry_robot_hvl/meshes/support_arch_v2.stl" scale="0.001 0.001 0.001"/>
+          <mesh filename="package://gantry_robot_hvl/meshes/support_arch_v2.stl" scale="${support_scale_x} ${support_scale_y} ${support_scale_z}"/>
         </geometry>
       </visual>
@@ -72,11 +78,11 @@
   <link name="h_beam_link">
         <visual>
-          <origin xyz="-5.5 -0.5 0.5" rpy="0 0 0"/>
+          <origin xyz="-2.6 -0.25 0.25" rpy="0 0 0"/>
           <geometry>
-            <mesh filename="package://gantry_robot_hvl/meshes/H-Beam_v3.stl" scale="1 1 1"/>
+            <mesh filename="package://gantry_robot_hvl/meshes/H-Beam_v3.stl" scale="${low_scale} ${low_scale} ${low_scale}"/>
           </geometry>
         </visual>
         <collision>
-          <origin xyz="-5.5 0 0.1" rpy="0 0 0"/>
+          <origin xyz="-2.6 0 0.05" rpy="0 0 0"/>
           <geometry>
             <box size="${h_beam_length} ${h_beam_width} ${h_beam_height}"/>
@@ -84,5 +90,5 @@
         </collision>
         <inertial>
-          <origin xyz="-5.5 0 0.1" rpy="0 0 0"/>
+          <origin xyz="-2.6 0 0.05" rpy="0 0 0"/>
           <mass value="${h_beam_mass}"/>
           <inertia
@@ -94,5 +100,5 @@
         <!-- ====================== H-Beam left joint ============================== -->
   <joint name="h_beam_joint_left" type="prismatic">
-          <origin xyz="0 0 4.5" rpy="0 0 0"/>
+          <origin xyz="0 0 3.1" rpy="0 0 0"/>
           <parent link="left_support_arch_link"/>
           <child link="h_beam_link"/>
@@ -100,10 +106,14 @@
           <calibration rising="0.0"/>
           <dynamics damping="0.0" friction="1.0"/>
-          <limit effort="30" velocity="1.0" lower="-4" upper="4" />
-          <safety_controller k_velocity="10" k_position="15" soft_lower_limit="-3.5" soft_upper_limit="3.5" />
+          <limit effort="30" velocity="1.0" lower="-2" upper="2" />
+          <safety_controller k_velocity="10" k_position="15" soft_lower_limit="-1.75" soft_upper_limit="1.75" />
   </joint>
         <!-- H-beam wheels -->
-        <xacro:property name="wheel_width" value="0.2" />
-        <xacro:property name="wheel_radius" value="0.35" />
+        <xacro:property name="wheel_width" value="0.1" />
+        <xacro:property name="wheel_radius" value="0.175" />
+        <xacro:property name="wheel_x" value="0.1" />
+        <xacro:property name="wheel_x_right" value="-5.3" />
+        <xacro:property name="wheel_y" value="0.225" />
+        <xacro:property name="wheel_z" value="0.375" />
   <link name="front_left_wheel">
           <visual name="flw">
@@ -121,5 +131,5 @@
   </link>
   <joint type="fixed" name="front_left_wheel_joint">
-          <origin xyz="0 0.45 -0.75" rpy="1.57057 0 1.57057"/>
+          <origin xyz="${wheel_x} ${wheel_y} -${wheel_z}" rpy="1.57057 0 1.57057"/>
           <child link="front_left_wheel"/>
           <parent link="h_beam_link"/>
@@ -140,5 +150,5 @@
   </link>
   <joint type="fixed" name="back_left_wheel_joint">
-          <origin xyz="0 -0.45 -0.75" rpy="1.57057 0 1.57057"/>
+          <origin xyz="${wheel_x} -${wheel_y} -${wheel_z}" rpy="1.57057 0 1.57057"/>
           <child link="back_left_wheel"/>
           <parent link="h_beam_link"/>
@@ -159,5 +169,5 @@
   </link>
   <joint type="fixed" name="front_right_wheel_joint">
-          <origin xyz="-11 0.45 -0.75" rpy="1.57057 0 1.57057"/>
+          <origin xyz="${wheel_x_right} ${wheel_y} -${wheel_z}" rpy="1.57057 0 1.57057"/>
           <child link="front_right_wheel"/>
           <parent link="h_beam_link"/>
@@ -178,5 +188,5 @@
   </link>
   <joint type="fixed" name="back_right_wheel_joint">
-          <origin xyz="-11 -0.45 -0.75" rpy="1.57057 0 1.57057"/>
+          <origin xyz="${wheel_x_right} -${wheel_y} -${wheel_z}" rpy="1.57057 0 1.57057"/>
           <child link="back_right_wheel"/>
           <parent link="h_beam_link"/>
@@ -188,9 +198,12 @@
         <xacro:property name="trolly_density" value="1" />
         <xacro:property name="trolly_mass" value="${trolly_length*trolly_height*trolly_width*trolly_density}" />
+        <xacro:property name="trolly_x" value="-2.6" />
+        <xacro:property name="trolly_y" value="0" />
+        <xacro:property name="trolly_z" value="-0.375" />
   <link name="trolly_link">
           <visual>
             <origin xyz="0 0 0" rpy="0 0 0"/>
             <geometry>
-              <mesh filename="package://gantry_robot_hvl/meshes/trolly_v3.stl" scale="0.01 0.01 0.01"/>
+              <mesh filename="package://gantry_robot_hvl/meshes/trolly_v3.stl" scale="${mid_scale} ${mid_scale} ${mid_scale}"/>
             </geometry>
           </visual>
@@ -211,5 +224,5 @@
   </link>
   <joint name="trolly_joint" type="prismatic">
-            <origin xyz="-5.5 0 -0.75" rpy="0 0 1.57057"/>
+            <origin xyz="${trolly_x} ${trolly_y} ${trolly_z}" rpy="0 0 1.57057"/>
             <parent link="h_beam_link"/>
             <child link="trolly_link"/>
@@ -217,6 +230,6 @@
             <calibration rising="0.0"/>
             <dynamics damping="0.0" friction="1.0"/>
-            <limit effort="30" velocity="1.0" lower="-4" upper="4" />
-            <safety_controller k_velocity="10" k_position="15" soft_lower_limit="-3.5" soft_upper_limit="3.5" />
+            <limit effort="30" velocity="1.0" lower="-2" upper="2" />
+            <safety_controller k_velocity="10" k_position="15" soft_lower_limit="-1.75" soft_upper_limit="1.75" />
   </joint>
           <!-- ========================= Crane ======================-->
@@ -226,9 +239,12 @@
           <xacro:property name="crane_density" value="1" />
           <xacro:property name="crane_mass" value="${crane_length*crane_height*crane_width*crane_density}" />
+          <xacro:property name="crane_x" value="0" />
+          <xacro:property name="crane_y" value="0" />
+          <xacro:property name="crane_z" value="0" />
   <link name="crane_link">
             <visual>
               <origin xyz="0 0 0" rpy="1.57057 0 0"/>
               <geometry>
-                <mesh filename="package://gantry_robot_hvl/meshes/crane_v3.stl" scale="0.01 0.01 0.01"/>
+                <mesh filename="package://gantry_robot_hvl/meshes/crane_v3.stl" scale="${mid_scale} ${mid_scale} ${mid_scale}"/>
               </geometry>
             </visual>
@@ -255,6 +271,6 @@
               <calibration rising="0.0"/>
               <dynamics damping="0.0" friction="10.0"/>
-              <limit effort="30" velocity="1.0" lower="-1.6" upper="0" />
-              <safety_controller k_velocity="10" k_position="15" soft_lower_limit="-1.5" soft_upper_limit="0" />
+              <limit effort="30" velocity="1.0" lower="-1.1" upper="0" />
+              <safety_controller k_velocity="10" k_position="15" soft_lower_limit="-1" soft_upper_limit="0" />
   </joint>
             <!-- ========================transmission============================ -->
