Commit message: Add files via upload

File: gantry_robot_hvl/urdf/ur10_crane.urdf (robot description, URDF)
Before this commit: robot ur10_crane, 20 links, 19 joints
Links:
- link crane_link: geometry collision box size=0.7 0.5 0.05; visual mesh filename=package://gantry_robot_hvl/meshes/crane_v3.stl scale=0.005 0.005 0.005
- link h_beam_link: geometry collision box size=5 0.1 0.35; visual mesh filename=package://gantry_robot_hvl/meshes/H-Beam_v3.stl scale=0.5 0.5 0.5
- link left_support_arch_link: geometry collision box size=5 0.5 2.5; visual mesh filename=package://gantry_robot_hvl/meshes/support_arch_v2.stl scale=0.0005 0.0005 0.00075
- link right_support_arch_link: geometry collision box size=5 0.5 2.5; visual mesh filename=package://gantry_robot_hvl/meshes/support_arch_v2.stl scale=0.0005 0.0005 0.00075
- link trolly_link: geometry collision box size=0.6 1 0.05; visual mesh filename=package://gantry_robot_hvl/meshes/trolly_v3.stl scale=0.005 0.005 0.005
